File: driver_cplex_rp2040/panel_header.kicad_sch (KiCad schematic)
At the start: 4 parts, among them J1 Conn_01x05, J2 Conn_01x05, J3 Conn_01x05, J4 Conn_01x05

Commit message: Worked on footprint assignment for rp2040 single panel cplex design.
Parts:
- J3, J4: footprint (none) -> panel_custom:C_0402_1005Metric
Changed lines of the file:
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@@
       (effects (font (size 1.27 1.27)) (justify left))
     )
-    (property "Footprint" "" (at 173.355 61.595 0)
+    (property "Footprint" "panel_custom:C_0402_1005Metric" (at 173.355 61.595 0)
       (effects (font (size 1.27 1.27)) hide)
     )
@@
       (effects (font (size 1.27 1.27)) (justify left))
     )
-    (property "Footprint" "" (at 173.355 46.99 0)
+    (property "Footprint" "panel_custom:C_0402_1005Metric" (at 173.355 46.99 0)
       (effects (font (size 1.27 1.27)) hide)
     )

Commit message: Worked on layout.
Parts:
- J3, J4: footprint panel_custom:C_0402_1005Metric -> panel_custom:ConnRcpt_1x5_SMH-105-02-X-S
Connections:
- net +5V: now also J1.5 (Pin_5), J3.5 (Pin_5); no longer J1.1 (Pin_1), J3.1 (Pin_1)
- net CS0: now also J2.5 (Pin_5); no longer J2.1 (Pin_1)
- net CS1: now also J2.4 (Pin_4), J4.5 (Pin_5); no longer J2.2 (Pin_2), J4.1 (Pin_1)
- net CS2: now also J4.4 (Pin_4); no longer J4.2 (Pin_2)
- net CS4: now also J2.2 (Pin_2); no longer J2.4 (Pin_4)
- net CS5: now also J2.1 (Pin_1), J4.2 (Pin_2); no longer J2.5 (Pin_5), J4.4 (Pin_4)
- net GND: now also J1.4 (Pin_4), J3.4 (Pin_4); no longer J1.2 (Pin_2), J3.2 (Pin_2)
- net MISO: now also J1.1 (Pin_1), J3.1 (Pin_1); no longer J1.5 (Pin_5), J3.5 (Pin_5)
- net MOSI: now also J1.2 (Pin_2), J3.2 (Pin_2); no longer J1.4 (Pin_4), J3.4 (Pin_4)
Other:
- moved on the sheet: J1, J2
Changed lines of the file:
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@@
     (effects (font (size 1.27 1.27)) (justify left))
   )
-  (symbol (lib_id "Connector_Generic:Conn_01x05") (at 93.98 61.595 0) (mirror y) (unit 1)
-    (in_bom yes) (on_board yes) (dnp no) (fields_autoplaced)
-    (property "Reference" "J2" (at 91.44 60.96 0)
+  (symbol (lib_id "Connector_Generic:Conn_01x05") (at 93.98 61.595 180) (unit 1)
+    (in_bom yes) (on_board yes) (dnp no)
+    (property "Reference" "J2" (at 91.44 62.23 0)
       (effects (font (size 1.27 1.27)) (justify left))
     )
-    (property "Value" "Conn_01x05" (at 91.44 63.5 0)
+    (property "Value" "Conn_01x05" (at 91.44 59.69 0)
       (effects (font (size 1.27 1.27)) (justify left))
     )
@@
     )
   )
-  (symbol (lib_id "Connector_Generic:Conn_01x05") (at 173.355 61.595 0) (unit 1)
-    (in_bom yes) (on_board yes) (dnp no) (fields_autoplaced)
-    (property "Reference" "J4" (at 176.53 60.96 0)
+  (symbol (lib_id "Connector_Generic:Conn_01x05") (at 173.355 61.595 0) (mirror x) (unit 1)
+    (in_bom yes) (on_board yes) (dnp no)
+    (property "Reference" "J4" (at 176.53 62.23 0)
       (effects (font (size 1.27 1.27)) (justify left))
     )
-    (property "Value" "Conn_01x05" (at 176.53 63.5 0)
+    (property "Value" "Conn_01x05" (at 176.53 59.69 0)
       (effects (font (size 1.27 1.27)) (justify left))
     )
-    (property "Footprint" "panel_custom:C_0402_1005Metric" (at 173.355 61.595 0)
+    (property "Footprint" "panel_custom:ConnRcpt_1x5_SMH-105-02-X-S" (at 173.355 61.595 0)
       (effects (font (size 1.27 1.27)) hide)
     )
@@
     )
   )
-  (symbol (lib_id "Connector_Generic:Conn_01x05") (at 173.355 46.99 0) (unit 1)
-    (in_bom yes) (on_board yes) (dnp no) (fields_autoplaced)
-    (property "Reference" "J3" (at 175.895 46.355 0)
+  (symbol (lib_id "Connector_Generic:Conn_01x05") (at 173.355 46.99 0) (mirror x) (unit 1)
+    (in_bom yes) (on_board yes) (dnp no)
+    (property "Reference" "J3" (at 175.895 47.625 0)
       (effects (font (size 1.27 1.27)) (justify left))
     )
-    (property "Value" "Conn_01x05" (at 175.895 48.895 0)
+    (property "Value" "Conn_01x05" (at 175.895 45.085 0)
       (effects (font (size 1.27 1.27)) (justify left))
     )
-    (property "Footprint" "panel_custom:C_0402_1005Metric" (at 173.355 46.99 0)
+    (property "Footprint" "panel_custom:ConnRcpt_1x5_SMH-105-02-X-S" (at 173.355 46.99 0)
       (effects (font (size 1.27 1.27)) hide)
     )
@@
     )
   )
-  (symbol (lib_id "Connector_Generic:Conn_01x05") (at 93.98 46.99 0) (mirror y) (unit 1)
-    (in_bom yes) (on_board yes) (dnp no) (fields_autoplaced)
-    (property "Reference" "J1" (at 91.44 46.355 0)
+  (symbol (lib_id "Connector_Generic:Conn_01x05") (at 93.98 46.99 180) (unit 1)
+    (in_bom yes) (on_board yes) (dnp no)
+    (property "Reference" "J1" (at 91.44 47.625 0)
       (effects (font (size 1.27 1.27)) (justify left))
     )
-    (property "Value" "Conn_01x05" (at 91.44 48.895 0)
+    (property "Value" "Conn_01x05" (at 91.44 45.085 0)
       (effects (font (size 1.27 1.27)) (justify left))
     )
