File: driver_cplex_rp2040/level_shifter.kicad_sch (KiCad schematic)
At the start: 204 parts, among them Q1 PNP, Q10 NPN, Q11 PNP, Q12 NPN, Q13 PNP, Q14 NPN, Q15 PNP, Q16 NPN, Q17 PNP, Q18 NPN, Q19 PNP, Q2 NPN, Q20 NPN, Q21 PNP, Q22 NPN, Q23 PNP, Q24 NPN, Q25 PNP, Q26 NPN, Q27 PNP, Q28 NPN, Q29 PNP, Q3 PNP, Q30 NPN, Q31 PNP, Q32 NPN, Q33 PNP, Q34 NPN, Q35 PNP, Q36 NPN, Q37 PNP, Q38 NPN, Q39 PNP, Q4 NPN, Q40 NPN, Q41 PNP, Q42 NPN, Q43 PNP, Q44 NPN, Q45 PNP, Q46 NPN, Q47 PNP, Q48 NPN, Q49 PNP, Q5 PNP, Q50 NPN, Q51 PNP, Q52 NPN, Q53 PNP, Q54 NPN, Q55 PNP, Q56 NPN, Q57 PNP, Q58 NPN, Q59 PNP, Q6 NPN, Q60 NPN, Q61 PNP, Q62 NPN, Q63 PNP, Q64 NPN, Q65 PNP, Q66 NPN, Q67 PNP, Q68 NPN, Q7 PNP, Q8 NPN, Q9 PNP

Commit message: Worked on footprint assignment for rp2040 single panel cplex design.
Parts:
- removed Q1, Q11, Q13, Q15, Q17, Q19, Q21, Q23, Q25, Q27, Q29, Q3, Q31, Q33, Q35, Q37, Q39, Q41, Q43, Q45, Q47, Q49, Q5, Q51, Q53, Q55, Q57, Q59, Q61, Q63, Q65, Q67, Q7, Q9: PNP, symbol Simulation_SPICE:PNP
- removed Q10, Q12, Q14, Q16, Q18, Q2, Q20, Q22, Q24, Q26, Q28, Q30, Q32, Q34, Q36, Q38, Q4, Q40, Q42, Q44, Q46, Q48, Q50, Q52, Q54, Q56, Q58, Q6, Q60, Q62, Q64, Q66, Q68, Q8: NPN, symbol Simulation_SPICE:NPN
- added Q1, Q10, Q11, Q12, Q13, Q14, Q15, Q16, Q17, Q18, Q19, Q2, Q20, Q21, Q22, Q23, Q24, Q25, Q26, Q27, Q28, Q29, Q3, Q30, Q31, Q32, Q33, Q34, Q4, Q5, Q6, Q7, Q8, Q9: 1xPNP and 1xNPN, panel_custom:SOT-963, symbol panel_custom:NST3946DP6T5G
- R10: renamed from R13; footprint (none) -> panel_custom:R_0201_0603Metric
- R100: renamed from R119; footprint (none) -> panel_custom:R_0201_0603Metric
- R101: renamed from R120; footprint (none) -> panel_custom:R_0201_0603Metric
- R102: renamed from R121; footprint (none) -> panel_custom:R_0201_0603Metric
- R103: renamed from R122; footprint (none) -> panel_custom:R_0201_0603Metric
- R104: renamed from R123; footprint (none) -> panel_custom:R_0201_0603Metric
- R105: renamed from R124; footprint (none) -> panel_custom:R_0201_0603Metric
- R106: renamed from R125; footprint (none) -> panel_custom:R_0201_0603Metric
- R107: renamed from R126; footprint (none) -> panel_custom:R_0201_0603Metric
- R108: renamed from R127; footprint (none) -> panel_custom:R_0201_0603Metric
- R109: renamed from R128; footprint (none) -> panel_custom:R_0201_0603Metric
- R11: renamed from R14; footprint (none) -> panel_custom:R_0201_0603Metric
- R110: renamed from R129; footprint (none) -> panel_custom:R_0201_0603Metric
- R111: renamed from R130; footprint (none) -> panel_custom:R_0201_0603Metric
- R112: renamed from R131; footprint (none) -> panel_custom:R_0201_0603Metric
- R113: renamed from R132; footprint (none) -> panel_custom:R_0201_0603Metric
- R114: renamed from R133; footprint (none) -> panel_custom:R_0201_0603Metric
- R115: renamed from R134; footprint (none) -> panel_custom:R_0201_0603Metric
- R116: renamed from R135; footprint (none) -> panel_custom:R_0201_0603Metric
- R117: renamed from R136; footprint (none) -> panel_custom:R_0201_0603Metric
- R118: renamed from R137; footprint (none) -> panel_custom:R_0201_0603Metric
- R119: renamed from R138; footprint (none) -> panel_custom:R_0201_0603Metric
- R12: renamed from R15; footprint (none) -> panel_custom:R_0201_0603Metric
- R120: renamed from R139; footprint (none) -> panel_custom:R_0201_0603Metric
- R121: renamed from R140; footprint (none) -> panel_custom:R_0201_0603Metric
- R122: renamed from R141; footprint (none) -> panel_custom:R_0201_0603Metric
- R123: renamed from R142; footprint (none) -> panel_custom:R_0201_0603Metric
- R124: renamed from R143; footprint (none) -> panel_custom:R_0201_0603Metric
- R125: renamed from R144; footprint (none) -> panel_custom:R_0201_0603Metric
- R126: renamed from R145; footprint (none) -> panel_custom:R_0201_0603Metric
- R127: renamed from R146; footprint (none) -> panel_custom:R_0201_0603Metric
- R128: renamed from R147; footprint (none) -> panel_custom:R_0201_0603Metric
- R129: renamed from R148; footprint (none) -> panel_custom:R_0201_0603Metric
- R13: renamed from R16; footprint (none) -> panel_custom:R_0201_0603Metric
- R130: renamed from R149; footprint (none) -> panel_custom:R_0201_0603Metric
- R131: renamed from R150; footprint (none) -> panel_custom:R_0201_0603Metric
- R132: renamed from R151; footprint (none) -> panel_custom:R_0201_0603Metric
- R133: renamed from R152; footprint (none) -> panel_custom:R_0201_0603Metric
- R134: renamed from R153; footprint (none) -> panel_custom:R_0201_0603Metric
- R135: renamed from R154; footprint (none) -> panel_custom:R_0201_0603Metric
- R136: renamed from R155; footprint (none) -> panel_custom:R_0201_0603Metric
- R137: renamed from R156; footprint (none) -> panel_custom:R_0201_0603Metric
- R138: renamed from R157; footprint (none) -> panel_custom:R_0201_0603Metric
- R139: renamed from R158; footprint (none) -> panel_custom:R_0201_0603Metric
- R14: renamed from R17; footprint (none) -> panel_custom:R_0201_0603Metric
- R140: renamed from R159; footprint (none) -> panel_custom:R_0201_0603Metric
- R141: renamed from R160; footprint (none) -> panel_custom:R_0201_0603Metric
- R15: renamed from R18; footprint (none) -> panel_custom:R_0201_0603Metric
- R16: renamed from R19; footprint (none) -> panel_custom:R_0201_0603Metric
- R17: renamed from R20; footprint (none) -> panel_custom:R_0201_0603Metric
- R18: renamed from R21; footprint (none) -> panel_custom:R_0201_0603Metric
- R19: renamed from R22; footprint (none) -> panel_custom:R_0201_0603Metric
- R20: renamed from R23; footprint (none) -> panel_custom:R_0201_0603Metric
- R21: renamed from R24; footprint (none) -> panel_custom:R_0201_0603Metric
- R22: renamed from R25; footprint (none) -> panel_custom:R_0201_0603Metric
- R23: renamed from R26; footprint (none) -> panel_custom:R_0201_0603Metric
- R24: renamed from R27; footprint (none) -> panel_custom:R_0201_0603Metric
- R25: renamed from R28; footprint (none) -> panel_custom:R_0201_0603Metric
- R26: renamed from R29; footprint (none) -> panel_custom:R_0201_0603Metric
- R27: renamed from R30; footprint (none) -> panel_custom:R_0201_0603Metric
- R28: renamed from R31; footprint (none) -> panel_custom:R_0201_0603Metric
- R29: renamed from R32; footprint (none) -> panel_custom:R_0201_0603Metric
- R30: renamed from R33; footprint (none) -> panel_custom:R_0201_0603Metric
- R31: renamed from R34; footprint (none) -> panel_custom:R_0201_0603Metric
- R32: renamed from R35; footprint (none) -> panel_custom:R_0201_0603Metric
- R33: renamed from R36; footprint (none) -> panel_custom:R_0201_0603Metric
- R34: renamed from R37; footprint (none) -> panel_custom:R_0201_0603Metric
- R35: renamed from R38; footprint (none) -> panel_custom:R_0201_0603Metric
- R36: renamed from R39; footprint (none) -> panel_custom:R_0201_0603Metric
- R37: renamed from R40; footprint (none) -> panel_custom:R_0201_0603Metric
- R38: renamed from R41; footprint (none) -> panel_custom:R_0201_0603Metric
- R39: renamed from R42; footprint (none) -> panel_custom:R_0201_0603Metric
- R40: renamed from R43; footprint (none) -> panel_custom:R_0201_0603Metric
- R41: renamed from R44; footprint (none) -> panel_custom:R_0201_0603Metric
- R42: renamed from R45; footprint (none) -> panel_custom:R_0201_0603Metric
- R43: renamed from R46; footprint (none) -> panel_custom:R_0201_0603Metric
- R44: renamed from R47; footprint (none) -> panel_custom:R_0201_0603Metric
- R45: renamed from R48; footprint (none) -> panel_custom:R_0201_0603Metric
- R46: renamed from R49; footprint (none) -> panel_custom:R_0201_0603Metric
- R47: renamed from R50; footprint (none) -> panel_custom:R_0201_0603Metric
- R48: renamed from R51; footprint (none) -> panel_custom:R_0201_0603Metric
- R49: renamed from R52; footprint (none) -> panel_custom:R_0201_0603Metric
- R50: renamed from R53; footprint (none) -> panel_custom:R_0201_0603Metric
- R51: renamed from R54; footprint (none) -> panel_custom:R_0201_0603Metric
- R52: renamed from R55; footprint (none) -> panel_custom:R_0201_0603Metric
- R53: renamed from R56; footprint (none) -> panel_custom:R_0201_0603Metric
- R54: renamed from R57; footprint (none) -> panel_custom:R_0201_0603Metric
- R55: renamed from R58; footprint (none) -> panel_custom:R_0201_0603Metric
- R56: renamed from R59; footprint (none) -> panel_custom:R_0201_0603Metric
- R57: renamed from R60; footprint (none) -> panel_custom:R_0201_0603Metric
- R58: renamed from R61; footprint (none) -> panel_custom:R_0201_0603Metric
- R59: renamed from R62; footprint (none) -> panel_custom:R_0201_0603Metric
- R6: renamed from R9; footprint (none) -> panel_custom:R_0201_0603Metric
- R60: renamed from R63; footprint (none) -> panel_custom:R_0201_0603Metric
- R61: renamed from R64; footprint (none) -> panel_custom:R_0201_0603Metric
- R62: renamed from R65; footprint (none) -> panel_custom:R_0201_0603Metric
- R63: renamed from R66; footprint (none) -> panel_custom:R_0201_0603Metric
- R64: renamed from R67; footprint (none) -> panel_custom:R_0201_0603Metric
- R65: renamed from R68; footprint (none) -> panel_custom:R_0201_0603Metric
- R66: renamed from R69; footprint (none) -> panel_custom:R_0201_0603Metric
- R67: renamed from R70; footprint (none) -> panel_custom:R_0201_0603Metric
- R68: renamed from R71; footprint (none) -> panel_custom:R_0201_0603Metric
- R69: renamed from R72; footprint (none) -> panel_custom:R_0201_0603Metric
- R7: renamed from R10; footprint (none) -> panel_custom:R_0201_0603Metric
- R70: renamed from R73; footprint (none) -> panel_custom:R_0201_0603Metric
- R71: renamed from R74; footprint (none) -> panel_custom:R_0201_0603Metric
- R72: renamed from R75; footprint (none) -> panel_custom:R_0201_0603Metric
- R73: renamed from R76; footprint (none) -> panel_custom:R_0201_0603Metric
- R74: renamed from R77; footprint (none) -> panel_custom:R_0201_0603Metric
- R75: renamed from R78; footprint (none) -> panel_custom:R_0201_0603Metric
- R76: renamed from R79; footprint (none) -> panel_custom:R_0201_0603Metric
- R77: renamed from R80; footprint (none) -> panel_custom:R_0201_0603Metric
- R78: renamed from R81; footprint (none) -> panel_custom:R_0201_0603Metric
- R79: renamed from R82; footprint (none) -> panel_custom:R_0201_0603Metric
- R8: renamed from R11; footprint (none) -> panel_custom:R_0201_0603Metric
- R80: renamed from R83; footprint (none) -> panel_custom:R_0201_0603Metric
- R81: renamed from R84; footprint (none) -> panel_custom:R_0201_0603Metric
- R82: renamed from R85; footprint (none) -> panel_custom:R_0201_0603Metric
- R83: renamed from R86; footprint (none) -> panel_custom:R_0201_0603Metric
- R84: renamed from R87; footprint (none) -> panel_custom:R_0201_0603Metric
- R85: renamed from R88; footprint (none) -> panel_custom:R_0201_0603Metric
- R86: renamed from R89; footprint (none) -> panel_custom:R_0201_0603Metric
- R87: renamed from R90; footprint (none) -> panel_custom:R_0201_0603Metric
- R88: renamed from R91; footprint (none) -> panel_custom:R_0201_0603Metric
- R89: renamed from R92; footprint (none) -> panel_custom:R_0201_0603Metric
- R9: renamed from R12; footprint (none) -> panel_custom:R_0201_0603Metric
- R90: renamed from R93; footprint (none) -> panel_custom:R_0201_0603Metric
- R91: renamed from R94; footprint (none) -> panel_custom:R_0201_0603Metric
- R92: renamed from R95; footprint (none) -> panel_custom:R_0201_0603Metric
- R93: renamed from R96; footprint (none) -> panel_custom:R_0201_0603Metric
- R94: renamed from R97; footprint (none) -> panel_custom:R_0201_0603Metric
- R95: renamed from R98; footprint (none) -> panel_custom:R_0201_0603Metric
- R96: renamed from R99; footprint (none) -> panel_custom:R_0201_0603Metric
- R97: renamed from R100; footprint (none) -> panel_custom:R_0201_0603Metric
- R98: renamed from R101; footprint (none) -> panel_custom:R_0201_0603Metric
- R99: renamed from R118; footprint (none) -> panel_custom:R_0201_0603Metric
Connections:
- net +5V: now also Q10.4, Q12.4, Q14.4, Q16.4, Q18.4, Q2.4, Q20.4, Q22.4, Q24.4, Q26.4, Q28.4, Q30.4, Q32.4, Q34.4, Q4.4, Q6.4, Q8.4
- net CP_5V_00: now also Q2.3, Q2.6
- net CP_5V_01: now also Q4.3, Q4.6
- net CP_5V_02: now also Q6.3, Q6.6
- net CP_5V_03: now also Q8.3, Q8.6
- net CP_5V_04: now also Q10.3, Q10.6
- net CP_5V_05: now also Q12.3, Q12.6
- net CP_5V_06: now also Q14.3, Q14.6
- net CP_5V_07: now also Q16.3, Q16.6
- net CP_5V_08: now also Q18.3, Q18.6
- net CP_5V_09: now also Q20.3, Q20.6
- net CP_5V_10: now also Q22.3, Q22.6
- net CP_5V_11: now also Q24.3, Q24.6
- net CP_5V_12: now also Q26.3, Q26.6
- net CP_5V_13: now also Q28.3, Q28.6
- net CP_5V_14: now also Q30.3, Q30.6
- net CP_5V_15: now also Q32.3, Q32.6
- net CP_5V_16: now also Q34.3, Q34.6
- net GND: now also Q10.1, Q12.1, Q14.1, Q16.1, Q18.1, Q2.1, Q20.1, Q22.1, Q24.1, Q26.1, Q28.1, Q30.1, Q32.1, Q34.1, Q4.1, Q6.1, Q8.1
- net at R18.2: now also Q3.4
- net at R59.1: now also Q13.1
- net at R80.2, R81.1: now also Q19.2
- net at R36.2: now also Q7.6, Q8.5
- net at R136.2, R137.1: now also Q33.2
- net at R76.2: now also Q17.6, Q18.5
- net at R69.1: now also Q15.3, Q16.2
- net at R62.2, R63.1: now also Q15.5
- net at R66.2: now also Q15.4
- net at R37.1: now also Q7.3, Q8.2
- net at R86.2, R87.1: now also Q21.5
- net at R44.2: now also Q10.5, Q9.6
- net at R40.2, R41.1: now also Q9.2
- net at R43.1: now also Q9.1
- net at R26.2: now also Q5.4
- net at R128.2, R129.1: now also Q31.2
- net at R24.2, R25.1: now also Q5.2
- net at R60.2: now also Q13.6, Q14.5
- net at R56.2, R57.1: now also Q13.2
- net at R53.1: now also Q11.3, Q12.2
- net at R29.1: now also Q5.3, Q6.2
- net at R117.1: now also Q27.3, Q28.2
- net at R85.1: now also Q19.3, Q20.2
- net at R83.1: now also Q19.1
- net at R38.2, R39.1: now also Q9.5
- net at R92.2: now also Q21.6, Q22.5
- net at R12.2: now also Q1.6, Q2.5
- net at R8.2, R9.1: now also Q1.2
- net at R11.1: now also Q1.1
- net at R120.2, R121.1: now also Q29.2
- net at R124.2: now also Q29.6, Q30.5
- net at R133.1: now also Q31.3, Q32.2
- net at R100.2: now also Q23.6, Q24.5
- net at R52.2: now also Q11.6, Q12.5
- net at R94.2, R95.1: now also Q23.5
- net at R130.2: now also Q31.4
- net at R72.2, R73.1: now also Q17.2
- net at R93.1: now also Q21.3, Q22.2
- net at R77.1: now also Q17.3, Q18.2
- net at R70.2, R71.1: now also Q17.5
- net at R74.2: now also Q17.4
- net at R42.2: now also Q9.4
- net at R101.1: now also Q23.3, Q24.2
- net at R98.2: now also Q23.4
- net at R99.1: now also Q23.1
- net at R140.2: now also Q33.6, Q34.5
- net at R32.2, R33.1: now also Q7.2
- net at R35.1: now also Q7.1
- net at R64.2, R65.1: now also Q15.2
- net at R14.2, R15.1: now also Q3.5
- net at R90.2: now also Q21.4
- net at R22.2, R23.1: now also Q5.5
- net at R132.2: now also Q31.6, Q32.5
- net at R96.2, R97.1: now also Q23.2
- net at R45.1: now also Q10.2, Q9.3
- net at R88.2, R89.1: now also Q21.2
- net at R91.1: now also Q21.1
- net at R102.2, R103.1: now also Q25.5
- net at R104.2, R105.1: now also Q25.2
- net at R13.1: now also Q1.3, Q2.2
- net at R48.2, R49.1: now also Q11.2
- net at R51.1: now also Q11.1
- net at R61.1: now also Q13.3, Q14.2
- net at R118.2, R119.1: now also Q29.5
- net at R131.1: now also Q31.1
- net at R68.2: now also Q15.6, Q16.5
- net at R67.1: now also Q15.1
- net at R110.2, R111.1: now also Q27.5
- net at R114.2: now also Q27.4
- net at R122.2: now also Q29.4
- net at R46.2, R47.1: now also Q11.5
- net at R50.2: now also Q11.4
- net at R16.2, R17.1: now also Q3.2
- net at R27.1: now also Q5.1
- net at R112.2, R113.1: now also Q27.2
- net at R20.2: now also Q3.6, Q4.5
- net at R30.2, R31.1: now also Q7.5
- net at R34.2: now also Q7.4
- net at R116.2: now also Q27.6, Q28.5
- net at R115.1: now also Q27.1
- net at R123.1: now also Q29.1
- net at R78.2, R79.1: now also Q19.5
- net at R109.1: now also Q25.3, Q26.2
- net at R106.2: now also Q25.4
- net at R141.1: now also Q33.3, Q34.2
- net at R107.1: now also Q25.1
- net at R28.2: now also Q5.6, Q6.5
- net at R19.1: now also Q3.1
- net at R108.2: now also Q25.6, Q26.5
- net at R54.2, R55.1: now also Q13.5
- net at R139.1: now also Q33.1
- net at R126.2, R127.1: now also Q31.5
- net at R6.2, R7.1: now also Q1.5
- net at R82.2: now also Q19.4
- net at R10.2: now also Q1.4
- net at R138.2: now also Q33.4
- net at R125.1: now also Q29.3, Q30.2
- net at R75.1: now also Q17.1
- net at R21.1: now also Q3.3, Q4.2
- net at R58.2: now also Q13.4
- net at R134.2, R135.1: now also Q33.5
- net at R84.2: now also Q19.6, Q20.5
Other:
- note added: "Maybe these? SOT-963 https://www.digikey.com/en/products/detail/onsemi/NST3946DP6T5G/1961256 SOT-563 https://www.digikey.com/en/products/detail/nexperia-usa-inc/PMBT3946VPN-115/2229323 SOT-363 https://www.lcsc.com/product-detail/Bipolar-span-style-background-color-ff0-Transistors-span-BJT_Diodes-Incorporated-MMDT2227-7-F_C191919.html"

Commit message: Worked on layout.
Connections:
- net CP_5V_00: now also Q1.6; no longer Q2.6
- net CP_5V_01: now also Q3.6; no longer Q4.6
- net CP_5V_02: now also Q5.6; no longer Q6.6
- net CP_5V_03: now also Q7.6; no longer Q8.6
- net CP_5V_04: now also Q9.6; no longer Q10.6
- net CP_5V_05: now also Q11.6; no longer Q12.6
- net CP_5V_06: now also Q13.6; no longer Q14.6
- net CP_5V_07: now also Q15.6; no longer Q16.6
- net CP_5V_08: now also Q17.6; no longer Q18.6
- net CP_5V_09: now also Q19.6; no longer Q20.6
- net CP_5V_10: now also Q21.6; no longer Q22.6
- net CP_5V_11: now also Q23.6; no longer Q24.6
- net CP_5V_12: now also Q25.6; no longer Q26.6
- net CP_5V_13: now also Q27.6; no longer Q28.6
- net CP_5V_14: now also Q29.6; no longer Q30.6
- net CP_5V_15: now also Q31.6; no longer Q32.6
- net CP_5V_16: now also Q33.6; no longer Q34.6
- net GND: now also Q1.1, Q11.1, Q13.1, Q15.1, Q17.1, Q19.1, Q21.1, Q23.1, Q25.1, Q27.1, Q29.1, Q3.1, Q31.1, Q33.1, Q5.1, Q7.1, Q9.1; no longer Q10.1, Q12.1, Q14.1, Q16.1, Q18.1, Q2.1, Q20.1, Q22.1, Q24.1, Q26.1, Q28.1, Q30.1, Q32.1, Q34.1, Q4.1, Q6.1, Q8.1
- net at Q3.3, R21.1: now also Q3.2; no longer Q4.2
- net at R59.1: now also Q14.1; no longer Q13.1
- net at R80.2, R81.1: now also Q20.2; no longer Q19.2
- net at R136.2, R137.1: now also Q34.2; no longer Q33.2
- net at Q21.3, R93.1: now also Q21.2; no longer Q22.2
- net at R99.1: now also Q24.1; no longer Q23.1
- net at R96.2, R97.1: now also Q24.2; no longer Q23.2
- net at Q24.5, R100.2: now also Q24.6; no longer Q23.6
- net at R107.1: now also Q26.1; no longer Q25.1
- net at R104.2, R105.1: now also Q26.2; no longer Q25.2
- net at Q26.5, R108.2: now also Q26.6; no longer Q25.6
- net at Q18.5, R76.2: now also Q18.6; no longer Q17.6
- net at Q7.3, R37.1: now also Q7.2; no longer Q8.2
- net at Q4.5, R20.2: now also Q4.6; no longer Q3.6
- net at R128.2, R129.1: now also Q32.2; no longer Q31.2
- net at R24.2, R25.1: now also Q6.2; no longer Q5.2
- net at R43.1: now also Q10.1; no longer Q9.1
- net at R40.2, R41.1: now also Q10.2; no longer Q9.2
- net at Q10.5, R44.2: now also Q10.6; no longer Q9.6
- net at R19.1: now also Q4.1; no longer Q3.1
- net at R16.2, R17.1: now also Q4.2; no longer Q3.2
- net at Q8.5, R36.2: now also Q8.6; no longer Q7.6
- net at Q11.3, R53.1: now also Q11.2; no longer Q12.2
- net at Q19.3, R85.1: now also Q19.2; no longer Q20.2
- net at R83.1: now also Q20.1; no longer Q19.1
- net at R56.2, R57.1: now also Q14.2; no longer Q13.2
- net at R67.1: now also Q16.1; no longer Q15.1
- net at R64.2, R65.1: now also Q16.2; no longer Q15.2
- net at Q16.5, R68.2: now also Q16.6; no longer Q15.6
- net at R120.2, R121.1: now also Q30.2; no longer Q29.2
- net at Q15.3, R69.1: now also Q15.2; no longer Q16.2
- net at Q12.5, R52.2: now also Q12.6; no longer Q11.6
- net at Q14.5, R60.2: now also Q14.6; no longer Q13.6
- net at Q27.3, R117.1: now also Q27.2; no longer Q28.2
- net at Q23.3, R101.1: now also Q23.2; no longer Q24.2
- net at R72.2, R73.1: now also Q18.2; no longer Q17.2
- net at Q22.5, R92.2: now also Q22.6; no longer Q21.6
- net at Q13.3, R61.1: now also Q13.2; no longer Q14.2
- net at Q2.5, R12.2: now also Q2.6; no longer Q1.6
- net at Q31.3, R133.1: now also Q31.2; no longer Q32.2
- net at Q20.5, R84.2: now also Q20.6; no longer Q19.6
- net at R27.1: now also Q6.1; no longer Q5.1
- net at Q6.5, R28.2: now also Q6.6; no longer Q5.6
- net at Q32.5, R132.2: now also Q32.6; no longer Q31.6
- net at Q9.3, R45.1: now also Q9.2; no longer Q10.2
- net at R88.2, R89.1: now also Q22.2; no longer Q21.2
- net at R91.1: now also Q22.1; no longer Q21.1
- net at Q1.3, R13.1: now also Q1.2; no longer Q2.2
- net at R32.2, R33.1: now also Q8.2; no longer Q7.2
- net at R131.1: now also Q32.1; no longer Q31.1
- net at R115.1: now also Q28.1; no longer Q27.1
- net at R112.2, R113.1: now also Q28.2; no longer Q27.2
- net at Q28.5, R116.2: now also Q28.6; no longer Q27.6
- net at Q17.3, R77.1: now also Q17.2; no longer Q18.2
- net at R123.1: now also Q30.1; no longer Q29.1
- net at R48.2, R49.1: now also Q12.2; no longer Q11.2
- net at Q33.3, R141.1: now also Q33.2; no longer Q34.2
- net at Q25.3, R109.1: now also Q25.2; no longer Q26.2
- net at R139.1: now also Q34.1; no longer Q33.1
- net at R35.1: now also Q8.1; no longer Q7.1
- net at Q29.3, R125.1: now also Q29.2; no longer Q30.2
- net at Q34.5, R140.2: now also Q34.6; no longer Q33.6
- net at R8.2, R9.1: now also Q2.2; no longer Q1.2
- net at R75.1: now also Q18.1; no longer Q17.1
- net at R11.1: now also Q2.1; no longer Q1.1
- net at Q30.5, R124.2: now also Q30.6; no longer Q29.6
- net at R51.1: now also Q12.1; no longer Q11.1
- net at Q5.3, R29.1: now also Q5.2; no longer Q6.2
Other:
- note added: "PNP + NPN array SOT-963 https://www.digikey.com/en/products/detail/onsemi/NST3946DP6T5G/1961256 PNP + NPN alternatives? SOT-563 https://www.digikey.com/en/products/detail/nexperia-usa-inc/PMBT3946VPN-115/2229323 SOT-363 https://www.lcsc.com/product-detail/Bipolar-span-style-background-color-ff0-Transistors-span-BJT_Diodes-Incorporated-MMDT2227-7-F_C191919.html"
- note added: "SWAPPED B's"
- note removed: "Maybe these? SOT-963 https://www.digikey.com/en/products/detail/onsemi/NST3946DP6T5G/1961256 SOT-563 https://www.digikey.com/en/products/detail/nexperia-usa-inc/PMBT3946VPN-115/2229323 SOT-363 https://www.lcsc.com/product-detail/Bipolar-span-style-background-color-ff0-Transistors-span-BJT_Diodes-Incorporated-MMDT2227-7-F_C191919.html"
- moved on the sheet: Q10B, Q11B, Q12B, Q13B, Q14B, Q15B, Q16B, Q17B, Q18B, Q19B, Q1B, Q20B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

Commit message: Worked on production files.
Parts:
- R10, R106, R107, R11, R114, R115, R122, R123, R130, R131, R138, R139, R18, R19, R26, R27, R34, R35, R42, R43, R50, R51, R58, R59, R66, R67, R74, R75, R82, R83, R90, R91, R98, R99: value 330 -> 100
- R100, R101, R108, R109, R116, R117, R12, R124, R125, R13, R132, R133, R140, R141, R20, R21, R28, R29, R36, R37, R44, R45, R52, R53, R60, R61, R68, R69, R76, R77, R84, R85, R92, R93: value 1k -> 2k
- R102, R110, R118, R126, R134, R14, R22, R30, R38, R46, R54, R6, R62, R70, R78, R86, R94: value 10 -> 10k
Other:
- note removed: "SWAPPED B's"
