File: spice/bjt_sim/npn/npn.kicad_sch (KiCad schematic)
At the start: 3 parts, among them Q1 NPN

Commit message: Worked on production files.
Parts:
- removed IE1: 20m, symbol Simulation_SPICE:IDC
- added R1, R2: 0.01, symbol Device:R
- added VCE1: 1, symbol Simulation_SPICE:VDC
- IB1: value 1m -> 250u
Connections:
- net 0: now also VCE1.1
- net at IB1.2: now also R2.1; no longer Q1.2 (B)
- net VCE: no longer names the net of Q1.1 (C)
- net VCE: now also R1.2
- new net: R1.1, VCE1.2
- new net Vb: Q1.2 (B), R2.2
Other:
- note added: ".dc VCE1 0 2 0.01 IB1 250u 3000u 250u"
- note removed: ".dc IB1 0.2m 5m 0.001m"
Changed lines of the file:
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@@
   (junction (at 95.25 83.82) (diameter 0) (color 0 0 0 0)
   )
-  (wire (pts (xy 128.905 65.405) (xy 95.25 65.405))
-    (stroke (width 0) (type default))
-  )
-  (wire (pts (xy 110.49 83.82) (xy 121.285 83.82))
+  (wire (pts (xy 128.905 55.245) (xy 95.25 55.245))
+    (stroke (width 0) (type default))
+  )
+  (wire (pts (xy 128.905 66.675) (xy 128.905 68.58))
+    (stroke (width 0) (type default))
+  )
+  (wire (pts (xy 119.38 83.82) (xy 121.285 83.82))
     (stroke (width 0) (type default))
   )
@@
     (stroke (width 0) (type default))
   )
-  (wire (pts (xy 95.25 65.405) (xy 95.25 83.82))
+  (wire (pts (xy 95.25 55.245) (xy 95.25 83.82))
+    (stroke (width 0) (type default))
+  )
+  (wire (pts (xy 128.905 55.245) (xy 128.905 56.515))
+    (stroke (width 0) (type default))
+  )
+  (wire (pts (xy 128.905 76.2) (xy 128.905 78.74))
     (stroke (width 0) (type default))
   )
@@
     (stroke (width 0) (type default))
   )
-  (wire (pts (xy 128.905 75.565) (xy 128.905 78.74))
-    (stroke (width 0) (type default))
-  )
-  (text ".dc IB1 0.2m 5m 0.001m" (at 102.87 102.87 0)
+  (wire (pts (xy 110.49 83.82) (xy 111.76 83.82))
+    (stroke (width 0) (type default))
+  )
+  (text ".dc VCE1 0 2 0.01 IB1 250u 3000u 250u" (at 99.695 104.775 0)
     (effects (font (size 1.27 1.27)) (justify left bottom))
   )
-  (label "VCE" (at 128.905 78.74 0) (fields_autoplaced)
+  (label "Vb" (at 119.38 83.82 0) (fields_autoplaced)
     (effects (font (size 1.27 1.27)) (justify left bottom))
   )
+  (symbol (lib_id "Device:R") (at 128.905 72.39 0) (unit 1)
+    (in_bom yes) (on_board yes) (dnp no) (fields_autoplaced)
+    (property "Reference" "R1" (at 130.81 71.12 0)
+      (effects (font (size 1.27 1.27)) (justify left))
+    )
+    (property "Value" "0.01" (at 130.81 73.66 0)
+      (effects (font (size 1.27 1.27)) (justify left))
+    )
+    (property "Footprint" "" (at 127.127 72.39 90)
+      (effects (font (size 1.27 1.27)) hide)
+    )
+    (property "Datasheet" "~" (at 128.905 72.39 0)
+      (effects (font (size 1.27 1.27)) hide)
+    )
+    (pin "2")
+    (pin "1")
+    (instances
+      (project "npn"
+        (path "/551237e1-e494-4286-a664-e2b40f8a2509"
+          (reference "R1") (unit 1)
+        )
+      )
+    )
+  )
   (symbol (lib_id "Simulation_SPICE:0") (at 95.25 96.52 0) (unit 1)
     (in_bom yes) (on_board yes) (dnp no) (fields_autoplaced)
@@
     )
   )
+  (symbol (lib_id "Simulation_SPICE:VDC") (at 128.905 61.595 0) (unit 1)
+    (in_bom yes) (on_board yes) (dnp no) (fields_autoplaced)
+    (property "Reference" "VCE1" (at 133.35 60.1952 0)
+      (effects (font (size 1.27 1.27)) (justify left))
+    )
+    (property "Value" "1" (at 133.35 62.7352 0)
+      (effects (font (size 1.27 1.27)) (justify left))
+    )
+    (property "Footprint" "" (at 128.905 61.595 0)
+      (effects (font (size 1.27 1.27)) hide)
+    )
+    (property "Datasheet" "~" (at 128.905 61.595 0)
+      (effects (font (size 1.27 1.27)) hide)
+    )
+    (property "Sim.Pins" "1=+ 2=-" (at 128.905 61.595 0)
+      (effects (font (size 1.27 1.27)) hide)
+    )
+    (property "Sim.Type" "DC" (at 128.905 61.595 0)
+      (effects (font (size 1.27 1.27)) hide)
+    )
+    (property "Sim.Device" "V" (at 128.905 61.595 0)
+      (effects (font (size 1.27 1.27)) (justify left) hide)
+    )
+    (pin "2")
+    (pin "1")
+    (instances
+      (project "npn"
+        (path "/551237e1-e494-4286-a664-e2b40f8a2509"
+          (reference "VCE1") (unit 1)
+        )
+      )
+    )
+  )
   (symbol (lib_id "Simulation_SPICE:IDC") (at 105.41 83.82 90) (unit 1)
     (in_bom yes) (on_board yes) (dnp no) (fields_autoplaced)
@@
       (effects (font (size 1.27 1.27)))
     )
-    (property "Value" "1m" (at 105.41 78.74 90)
+    (property "Value" "250u" (at 105.41 78.74 90)
       (effects (font (size 1.27 1.27)))
     )
@@
     )
   )
-  (symbol (lib_id "Simulation_SPICE:IDC") (at 128.905 70.485 0) (unit 1)
-    (in_bom yes) (on_board yes) (dnp no) (fields_autoplaced)
-    (property "Reference" "IE1" (at 133.35 69.215 0)
-      (effects (font (size 1.27 1.27)) (justify left))
-    )
-    (property "Value" "20m" (at 133.35 71.755 0)
-      (effects (font (size 1.27 1.27)) (justify left))
-    )
-    (property "Footprint" "" (at 128.905 70.485 0)
-      (effects (font (size 1.27 1.27)) hide)
-    )
-    (property "Datasheet" "~" (at 128.905 70.485 0)
-      (effects (font (size 1.27 1.27)) hide)
-    )
-    (property "Sim.Pins" "1=+ 2=-" (at 128.905 70.485 0)
-      (effects (font (size 1.27 1.27)) hide)
-    )
-    (property "Sim.Type" "DC" (at 128.905 70.485 0)
-      (effects (font (size 1.27 1.27)) hide)
-    )
-    (property "Sim.Device" "I" (at 128.905 70.485 0)
-      (effects (font (size 1.27 1.27)) hide)
-    )
-    (pin "1")
-    (pin "2")
-    (instances
-      (project "npn"
-        (path "/551237e1-e494-4286-a664-e2b40f8a2509"
-          (reference "IE1") (unit 1)
-        )
-      )
+  (symbol (lib_id "Device:R") (at 115.57 83.82 90) (unit 1)
+    (in_bom yes) (on_board yes) (dnp no) (fields_autoplaced)
+    (property "Reference" "R2" (at 115.57 77.47 90)
+      (effects (font (size 1.27 1.27)))
+    )
+    (property "Value" "0.01" (at 115.57 80.01 90)
+      (effects (font (size 1.27 1.27)))
+    )
+    (property "Footprint" "" (at 115.57 85.598 90)
+      (effects (font (size 1.27 1.27)) hide)
+    )
+    (property "Datasheet" "~" (at 115.57 83.82 0)
+      (effects (font (size 1.27 1.27)) hide)
+    )
+    (pin "2")
+    (pin "1")
+    (instances
+      (project "npn"
+        (path "/551237e1-e494-4286-a664-e2b40f8a2509"
+          (reference "R2") (unit 1)
+        )
+      )
