File: driver_rp2350/panel_led.kicad_sch (KiCad schematic)
At the start: 272 parts

Commit message: Worked on rp2350 schematic.
Parts:
- renumbered D_70 to D_07, D_80 to D_08, D_90 to D_09, D_A0 to D_0A, D_B0 to D_0B, D_C0 to D_0C, D_D0 to D_0D, D_E0 to D_0E, D_F0 to D_0F, D_71 to D_17, D_81 to D_18, D_91 to D_19, D_A1 to D_1A, D_B1 to D_1B, D_C1 to D_1C, D_D1 to D_1D, D_E1 to D_1E, D_F1 to D_1F, D_72 to D_27, D_82 to D_28, D_92 to D_29, D_A2 to D_2A, D_B2 to D_2B, D_C2 to D_2C, D_D2 to D_2D, D_E2 to D_2E, D_F2 to D_2F, D_73 to D_37, D_83 to D_38, D_93 to D_39, D_A3 to D_3A, D_B3 to D_3B, D_C3 to D_3C, D_D3 to D_3D, D_E3 to D_3E, D_F3 to D_3F, D_74 to D_47, D_84 to D_48, D_94 to D_49, D_A4 to D_4A, D_B4 to D_4B, D_C4 to D_4C, D_D4 to D_4D, D_E4 to D_4E, D_F4 to D_4F, D_75 to D_57, D_85 to D_58, D_95 to D_59, D_A5 to D_5A, D_B5 to D_5B, D198 to D_5C, D214 to D_5D, D230 to D_5E, D246 to D_5F, D119 to D_67, D135 to D_68, D151 to D_69, D167 to D_6A, D183 to D_6B, D199 to D_6C, D215 to D_6D, D231 to D_6E, D247 to D_6F, D120 to D_77, D136 to D_78, D152 to D_79, D168 to D_7A, D184 to D_7B, D200 to D_7C, D216 to D_7D, D232 to D_7E, D248 to D_7F, D121 to D_87, D137 to D_88, D153 to D_89, D169 to D_8A, D185 to D_8B, D201 to D_8C, D217 to D_8D, D233 to D_8E, D249 to D_8F, D122 to D_97, D138 to D_98, D154 to D_99, D170 to D_9A, D186 to D_9B, D202 to D_9C, D218 to D_9D, D234 to D_9E, D250 to D_9F, D123 to D_A7, D139 to D_A8, D155 to D_A9, D171 to D_AA, D187 to D_AB, D203 to D_AC, D219 to D_AD, D235 to D_AE, D251 to D_AF, D124 to D_B7, D140 to D_B8, D156 to D_B9, D172 to D_BA, D188 to D_BB, D204 to D_BC, D220 to D_BD, D236 to D_BE, D252 to D_BF, D125 to D_C7, D141 to D_C8, D157 to D_C9, D173 to D_CA, D189 to D_CB, D205 to D_CC, D221 to D_CD, D237 to D_CE, D253 to D_CF, D126 to D_D7, D142 to D_D8, D158 to D_D9, D174 to D_DA, D190 to D_DB, D206 to D_DC, D222 to D_DD, D238 to D_DE, D254 to D_DF, D127 to D_E7, D143 to D_E8, D159 to D_E9, D175 to D_EA, D191 to D_EB, D207 to D_EC, D223 to D_ED, D239 to D_EE, D255 to D_EF, D128 to D_F7, D144 to D_F8, D160 to D_F9, D176 to D_FA, D192 to D_FB, D208 to D_FC, D224 to D_FD, D240 to D_FE, D256 to D_FF

Commit message: Worked on rp2350 schematic.
Parts:
- renumbered R102 to R1, R111 to R10, R112 to R11, R113 to R12, R114 to R13, R115 to R14, R116 to R15, R117 to R16, R103 to R2, R104 to R3, R105 to R4, R106 to R5, R107 to R6, R108 to R7, R109 to R8, R110 to R9
Changed lines of the file:
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@@
 	(generator_version "9.0")
 	(paper "User" 355.6 254)
-	(text "Note on LED naming:  \n\nD_XY  where X = row number, Y = col number\n\nrow and col numbers in {1, 2, 3, ..., A, B, C, D, E, F}"
+	(text "Note on LED naming:  \nD_XY  where X = row number, Y = col number\nrow and col numbers in {1, 2, 3, ..., A, B, C, D, E, F}"
 		(exclude_from_sim no)
 		(at 29.464 221.742 0)
@@
 		(dnp no)
 		(fields_autoplaced yes)
-		(property "Reference" "R105"
+		(property "Reference" "R4"
 			(at 86.36 52.0699 0)
 			(effects
@@
 			(project "panel"
 				(path "/1e634561-32a0-4ffa-9d4f-e93f355464d5/9e6027a1-8475-463d-b347-a287726616e8"
-					(reference "R105")
+					(reference "R4")
 					(unit 1)
 				)
@@
 		(dnp no)
 		(fields_autoplaced yes)
-		(property "Reference" "R104"
+		(property "Reference" "R3"
 			(at 68.58 52.0699 0)
 			(effects
@@
 			(project "panel"
 				(path "/1e634561-32a0-4ffa-9d4f-e93f355464d5/9e6027a1-8475-463d-b347-a287726616e8"
-					(reference "R104")
+					(reference "R3")
 					(unit 1)
 				)
@@
 		(dnp no)
 		(fields_autoplaced yes)
-		(property "Reference" "R109"
+		(property "Reference" "R8"
 			(at 157.48 52.0699 0)
 			(effects
@@
 			(project "panel"
 				(path "/1e634561-32a0-4ffa-9d4f-e93f355464d5/9e6027a1-8475-463d-b347-a287726616e8"
-					(reference "R109")
+					(reference "R8")
 					(unit 1)
 				)
@@
 		(dnp no)
 		(fields_autoplaced yes)
-		(property "Reference" "R116"
+		(property "Reference" "R15"
 			(at 281.305 52.0699 0)
 			(effects
@@
 			(project "panel"
 				(path "/1e634561-32a0-4ffa-9d4f-e93f355464d5/9e6027a1-8475-463d-b347-a287726616e8"
-					(reference "R116")
+					(reference "R15")
 					(unit 1)
 				)
@@
 		(dnp no)
 		(fields_autoplaced yes)
-		(property "Reference" "R115"
+		(property "Reference" "R14"
 			(at 263.525 52.0699 0)
 			(effects
@@
 			(project "panel"
 				(path "/1e634561-32a0-4ffa-9d4f-e93f355464d5/9e6027a1-8475-463d-b347-a287726616e8"
-					(reference "R115")
+					(reference "R14")
 					(unit 1)
 				)
@@
 		(dnp no)
 		(fields_autoplaced yes)
-		(property "Reference" "R112"
+		(property "Reference" "R11"
 			(at 210.185 52.0699 0)
 			(effects
@@
 			(project "panel"
 				(path "/1e634561-32a0-4ffa-9d4f-e93f355464d5/9e6027a1-8475-463d-b347-a287726616e8"
-					(reference "R112")
+					(reference "R11")
 					(unit 1)
 				)
@@
 		(dnp no)
 		(fields_autoplaced yes)
-		(property "Reference" "R113"
+		(property "Reference" "R12"
 			(at 227.965 52.0699 0)
 			(effects
@@
 			(project "panel"
 				(path "/1e634561-32a0-4ffa-9d4f-e93f355464d5/9e6027a1-8475-463d-b347-a287726616e8"
-					(reference "R113")
+					(reference "R12")
 					(unit 1)
 				)
@@
 		(dnp no)
 		(fields_autoplaced yes)
-		(property "Reference" "R107"
+		(property "Reference" "R6"
 			(at 121.92 52.0699 0)
 			(effects
@@
 			(project "panel"
 				(path "/1e634561-32a0-4ffa-9d4f-e93f355464d5/9e6027a1-8475-463d-b347-a287726616e8"
-					(reference "R107")
+					(reference "R6")
 					(unit 1)
 				)
@@
 		(dnp no)
 		(fields_autoplaced yes)
-		(property "Reference" "R110"
+		(property "Reference" "R9"
 			(at 174.625 52.0699 0)
 			(effects
@@
 			(project "panel"
 				(path "/1e634561-32a0-4ffa-9d4f-e93f355464d5/9e6027a1-8475-463d-b347-a287726616e8"
-					(reference "R110")
+					(reference "R9")
 					(unit 1)
 				)
@@
 		(dnp no)
 		(fields_autoplaced yes)
-		(property "Reference" "R102"
+		(property "Reference" "R1"
 			(at 33.02 52.0699 0)
 			(effects
@@
 			(project "panel"
 				(path "/1e634561-32a0-4ffa-9d4f-e93f355464d5/9e6027a1-8475-463d-b347-a287726616e8"
-					(reference "R102")
+					(reference "R1")
 					(unit 1)
 				)
@@
 		(dnp no)
 		(fields_autoplaced yes)
-		(property "Reference" "R111"
+		(property "Reference" "R10"
 			(at 192.405 52.0699 0)
 			(effects
@@
 			(project "panel"
 				(path "/1e634561-32a0-4ffa-9d4f-e93f355464d5/9e6027a1-8475-463d-b347-a287726616e8"
-					(reference "R111")
+					(reference "R10")
 					(unit 1)
 				)
@@
 		(dnp no)
 		(fields_autoplaced yes)
-		(property "Reference" "R106"
+		(property "Reference" "R5"
 			(at 104.14 52.0699 0)
 			(effects
@@
 			(project "panel"
 				(path "/1e634561-32a0-4ffa-9d4f-e93f355464d5/9e6027a1-8475-463d-b347-a287726616e8"
-					(reference "R106")
+					(reference "R5")
 					(unit 1)
 				)
@@
 		(dnp no)
 		(fields_autoplaced yes)
-		(property "Reference" "R103"
+		(property "Reference" "R2"
 			(at 50.8 52.0699 0)
 			(effects
@@
 			(project "panel"
 				(path "/1e634561-32a0-4ffa-9d4f-e93f355464d5/9e6027a1-8475-463d-b347-a287726616e8"
-					(reference "R103")
+					(reference "R2")
 					(unit 1)
 				)
@@
 		(dnp no)
 		(fields_autoplaced yes)
-		(property "Reference" "R114"
+		(property "Reference" "R13"
 			(at 245.745 52.0699 0)
 			(effects
@@
 			(project "panel"
 				(path "/1e634561-32a0-4ffa-9d4f-e93f355464d5/9e6027a1-8475-463d-b347-a287726616e8"
-					(reference "R114")
+					(reference "R13")
 					(unit 1)
 				)
@@
 		(dnp no)
 		(fields_autoplaced yes)
-		(property "Reference" "R117"
+		(property "Reference" "R16"
 			(at 299.085 52.0699 0)
 			(effects
@@
 			(project "panel"
 				(path "/1e634561-32a0-4ffa-9d4f-e93f355464d5/9e6027a1-8475-463d-b347-a287726616e8"
-					(reference "R117")
+					(reference "R16")
 					(unit 1)
 				)
@@
 		(dnp no)
 		(fields_autoplaced yes)
-		(property "Reference" "R108"
+		(property "Reference" "R7"
 			(at 139.7 52.0699 0)
 			(effects
@@
 			(project "panel"
 				(path "/1e634561-32a0-4ffa-9d4f-e93f355464d5/9e6027a1-8475-463d-b347-a287726616e8"
-					(reference "R108")
+					(reference "R7")
 					(unit 1)
 				)
