File: driver_rp2350/drivers.kicad_sch (KiCad schematic)
At the start: 0 parts

Commit message: Finished first version of schematic for rp2350 G6 panel.
Parts:
- added C22, C23, C24, C25, C26, C27, C28, C29, C30, C31, C32, C33, C34, C35, C36, C37, C38, C39, C40, C41, C42, C43, C44, C45, C46, C47, C48, C49, C50, C51, C52, C53: 100nF, symbol Device:C_Small
- added C54, C55, C56, C57, C58, C59, C60, C61: 10uF, symbol Device:C
- added U10, U11, U12, U13, U14, U15, U16, U17, U18, U19, U20, U21, U22, U23, U24, U25, U26, U27, U28, U29, U30, U31, U32, U33, U34, U35, U4, U5, U6, U7, U8, U9: UCC27517, symbol panel_custom:UCC27517
Connections:
- new net +5V: C22.1, C23.1, C24.1, C25.1, C26.1, C27.1, C28.1, C29.1, C30.1, C31.1, C32.1, C33.1, C34.1, C35.1, C36.1, C37.1, C38.1, C39.1, C40.1, C41.1, C42.1, C43.1, C44.1, C45.1, C46.1, C47.1, C48.1, C49.1, C50.1, C51.1, C52.1, C53.1, C54.1, C55.1, C56.1, C57.1, C58.1, C59.1, C60.1, C61.1, U10.1 (VDD), U11.1 (VDD), U12.1 (VDD), U13.1 (VDD), U14.1 (VDD), U15.1 (VDD), U16.1 (VDD), U17.1 (VDD), U18.1 (VDD), U19.1 (VDD), U20.1 (VDD), U21.1 (VDD), U22.1 (VDD), U23.1 (VDD), U24.1 (VDD), U25.1 (VDD), U26.1 (VDD), U27.1 (VDD), U28.1 (VDD), U29.1 (VDD), U30.1 (VDD), U31.1 (VDD), U32.1 (VDD), U33.1 (VDD), U34.1 (VDD), U35.1 (VDD), U4.1 (VDD), U5.1 (VDD), U6.1 (VDD), U7.1 (VDD), U8.1 (VDD), U9.1 (VDD)
- new net COL_0: U4.5 (OUT)
- new net COL_1: U5.5 (OUT)
- new net COL_2: U6.5 (OUT)
- new net COL_3: U7.5 (OUT)
- new net COL_4: U8.5 (OUT)
- new net COL_5: U9.5 (OUT)
- new net COL_6: U10.5 (OUT)
- new net COL_7: U11.5 (OUT)
- new net COL_8: U12.5 (OUT)
- new net COL_9: U13.5 (OUT)
- new net COL_A: U14.5 (OUT)
- new net COL_B: U15.5 (OUT)
- new net COL_C: U16.5 (OUT)
- new net COL_D: U17.5 (OUT)
- new net COL_E: U18.5 (OUT)
- new net COL_F: U19.5 (OUT)
- new net COL_MCU_0: U4.3 (IN+)
- new net COL_MCU_1: U5.3 (IN+)
- new net COL_MCU_2: U6.3 (IN+)
- new net COL_MCU_3: U7.3 (IN+)
- new net COL_MCU_4: U8.3 (IN+)
- new net COL_MCU_5: U9.3 (IN+)
- new net COL_MCU_6: U10.3 (IN+)
- new net COL_MCU_7: U11.3 (IN+)
- new net COL_MCU_8: U12.3 (IN+)
- new net COL_MCU_9: U13.3 (IN+)
- new net COL_MCU_A: U14.3 (IN+)
- new net COL_MCU_B: U15.3 (IN+)
- new net COL_MCU_C: U16.3 (IN+)
- new net COL_MCU_D: U17.3 (IN+)
- new net COL_MCU_E: U18.3 (IN+)
- new net COL_MCU_F: U19.3 (IN+)
- new net GND: C22.2, C23.2, C24.2, C25.2, C26.2, C27.2, C28.2, C29.2, C30.2, C31.2, C32.2, C33.2, C34.2, C35.2, C36.2, C37.2, C38.2, C39.2, C40.2, C41.2, C42.2, C43.2, C44.2, C45.2, C46.2, C47.2, C48.2, C49.2, C50.2, C51.2, C52.2, C53.2, C54.2, C55.2, C56.2, C57.2, C58.2, C59.2, C60.2, C61.2, U10.2 (GND), U10.4 (IN-), U11.2 (GND), U11.4 (IN-), U12.2 (GND), U12.4 (IN-), U13.2 (GND), U13.4 (IN-), U14.2 (GND), U14.4 (IN-), U15.2 (GND), U15.4 (IN-), U16.2 (GND), U16.4 (IN-), U17.2 (GND), U17.4 (IN-), U18.2 (GND), U18.4 (IN-), U19.2 (GND), U19.4 (IN-), U20.2 (GND), U20.4 (IN-), U21.2 (GND), U21.4 (IN-), U22.2 (GND), U22.4 (IN-), U23.2 (GND), U23.4 (IN-), U24.2 (GND), U24.4 (IN-), U25.2 (GND), U25.4 (IN-), U26.2 (GND), U26.4 (IN-), U27.2 (GND), U27.4 (IN-), U28.2 (GND), U28.4 (IN-), U29.2 (GND), U29.4 (IN-), U30.2 (GND), U30.4 (IN-), U31.2 (GND), U31.4 (IN-), U32.2 (GND), U32.4 (IN-), U33.2 (GND), U33.4 (IN-), U34.2 (GND), U34.4 (IN-), U35.2 (GND), U35.4 (IN-), U4.2 (GND), U4.4 (IN-), U5.2 (GND), U5.4 (IN-), U6.2 (GND), U6.4 (IN-), U7.2 (GND), U7.4 (IN-), U8.2 (GND), U8.4 (IN-), U9.2 (GND), U9.4 (IN-)
- new net ROW_0: U20.5 (OUT)
- new net ROW_1: U21.5 (OUT)
- new net ROW_2: U22.5 (OUT)
- new net ROW_3: U23.5 (OUT)
- new net ROW_4: U24.5 (OUT)
- new net ROW_5: U25.5 (OUT)
- new net ROW_6: U26.5 (OUT)
- new net ROW_7: U27.5 (OUT)
- new net ROW_8: U28.5 (OUT)
- new net ROW_9: U29.5 (OUT)
- new net ROW_A: U30.5 (OUT)
- new net ROW_B: U31.5 (OUT)
- new net ROW_C: U32.5 (OUT)
- new net ROW_D: U33.5 (OUT)
- new net ROW_E: U34.5 (OUT)
- new net ROW_F: U35.5 (OUT)
- new net ROW_MCU_0: U20.3 (IN+)
- new net ROW_MCU_1: U21.3 (IN+)
- new net ROW_MCU_2: U22.3 (IN+)
- new net ROW_MCU_3: U23.3 (IN+)
- new net ROW_MCU_4: U24.3 (IN+)
- new net ROW_MCU_5: U25.3 (IN+)
- new net ROW_MCU_6: U26.3 (IN+)
- new net ROW_MCU_7: U27.3 (IN+)
- new net ROW_MCU_8: U28.3 (IN+)
- new net ROW_MCU_9: U29.3 (IN+)
- new net ROW_MCU_A: U30.3 (IN+)
- new net ROW_MCU_B: U31.3 (IN+)
- new net ROW_MCU_C: U32.3 (IN+)
- new net ROW_MCU_D: U33.3 (IN+)
- new net ROW_MCU_E: U34.3 (IN+)
- new net ROW_MCU_F: U35.3 (IN+)
Other:
- note added: "Column Drivers"
- note added: "Row Drivers"
