File: driver_rp2350_old16x16/driver_rp2350.kicad_pcb (KiCad board)
At the start: 6 copper layers, 45 x 45 mm, 0 parts

Commit message: Worked on new 18x18 led version of rp2350 design.
Other:
- board outline removed
Changed lines of the file:
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@@
 	)
 	(net 0 "")
-	(gr_rect
-		(start 50 50)
-		(end 95 95)
-		(stroke
-			(width 0.25)
-			(type default)
-		)
-		(fill no)
-		(layer "Edge.Cuts")
-	)
 	(embedded_fonts no)
 )
