File: driver_rp2350_old16x16/drivers.kicad_sch (KiCad schematic)
At the start: 80 parts, among them U10 UCC27517, U11 UCC27517, U12 UCC27517, U13 UCC27517, U14 UCC27517, U15 UCC27517, U16 UCC27517, U17 UCC27517, U18 UCC27517, U19 UCC27517, U20 UCC27517, U21 UCC27517, U22 UCC27517, U23 UCC27517, U24 UCC27517, U25 UCC27517, U26 UCC27517, U27 UCC27517, U28 UCC27517, U29 UCC27517, U3 UCC27517, U30 UCC27517, U31 UCC27517, U32 UCC27517, U33 UCC27517, U34 UCC27517, U35 UCC27517, U36 UCC27517, U37 UCC27517, U38 UCC27517, U4 UCC27517, U5 UCC27517, U6 UCC27517, U7 UCC27517, U8 UCC27517, U9 UCC27517

Commit message: Worked on new 18x18 led version of rp2350 design.
Parts:
- removed C36, C37, C54, C55: 100nF, Capacitor_SMD:C_0402_1005Metric, symbol Device:C_Small
- removed U19, U20, U37, U38: UCC27517, symbol panel_custom:UCC27517
- C22: renamed from C20; footprint Capacitor_SMD:C_0402_1005Metric -> (none)
- C23: renamed from C21; footprint Capacitor_SMD:C_0402_1005Metric -> (none)
- C24: renamed from C22; footprint Capacitor_SMD:C_0402_1005Metric -> (none)
- C25: renamed from C23; footprint Capacitor_SMD:C_0402_1005Metric -> (none)
- C26: renamed from C24; footprint Capacitor_SMD:C_0402_1005Metric -> (none)
- C27: renamed from C25; footprint Capacitor_SMD:C_0402_1005Metric -> (none)
- C28: renamed from C26; footprint Capacitor_SMD:C_0402_1005Metric -> (none)
- C29: renamed from C27; footprint Capacitor_SMD:C_0402_1005Metric -> (none)
- C30: renamed from C28; footprint Capacitor_SMD:C_0402_1005Metric -> (none)
- C31: renamed from C29; footprint Capacitor_SMD:C_0402_1005Metric -> (none)
- C32: renamed from C30; footprint Capacitor_SMD:C_0402_1005Metric -> (none)
- C33: renamed from C31; footprint Capacitor_SMD:C_0402_1005Metric -> (none)
- C34: renamed from C32; footprint Capacitor_SMD:C_0402_1005Metric -> (none)
- C35: renamed from C33; footprint Capacitor_SMD:C_0402_1005Metric -> (none)
- C36: renamed from C34; footprint Capacitor_SMD:C_0402_1005Metric -> (none)
- C37: renamed from C35; footprint Capacitor_SMD:C_0402_1005Metric -> (none)
- C38, C39, C40, C41, C42, C43, C44, C45, C46, C47, C48, C49, C50, C51, C52, C53: footprint Capacitor_SMD:C_0402_1005Metric -> (none)
- C54: renamed from C56; footprint Capacitor_SMD:C_0402_1005Metric -> (none)
- C55: renamed from C57; footprint Capacitor_SMD:C_0402_1005Metric -> (none)
- C56: renamed from C58; footprint Capacitor_SMD:C_0402_1005Metric -> (none)
- C57: renamed from C59; footprint Capacitor_SMD:C_0402_1005Metric -> (none)
- C58: renamed from C60; footprint Capacitor_SMD:C_0402_1005Metric -> (none)
- C59: renamed from C61; footprint Capacitor_SMD:C_0402_1005Metric -> (none)
- C60: renamed from C62; footprint Capacitor_SMD:C_0402_1005Metric -> (none)
- C61: renamed from C63; footprint Capacitor_SMD:C_0402_1005Metric -> (none)
- renumbered U9 to U10, U10 to U11, U11 to U12, U12 to U13, U13 to U14, U14 to U15, U15 to U16, U16 to U17, U17 to U18, U18 to U19, U21 to U20, U22 to U21, U23 to U22, U24 to U23, U25 to U24, U26 to U25, U27 to U26, U28 to U27, U29 to U28, U30 to U29, U31 to U30, U32 to U31, U33 to U32, U34 to U33, U35 to U34, U36 to U35, U3 to U4, U4 to U5, U5 to U6, U6 to U7, U7 to U8, U8 to U9
Other:
- note removed: "Maybe use larger capacitance for 10uF capacitors (say 22uF) if using smaller package size components, e.g. 0402."
- moved on the sheet: C30, C31, C32, C33, C34, C35, C36, C37, C46, C47, C48, C49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
