File: driver_rp2350_old16x16/panel_mcu.kicad_sch (KiCad schematic)
At the start: 32 parts, among them SW1 SW_Push, SW2 SW_Push, U1 W25Q16JVUXIQ_TR, U2 RP2350_80QFN, Y1 ABM8-272-T3

Commit message: Worked on new 18x18 led version of rp2350 design.
Parts:
- C10: renamed from C8; value 4.7uF -> 4.7u
- C11: renamed from C9; value 100nF -> 100n
- C12: renamed from C10; value 100nF -> 100n
- C13: renamed from C11; value 100nF -> 100n
- C14: renamed from C12; value 100nF -> 100n
- C15: renamed from C13; value 100nF -> 100n
- C16: renamed from C14; value 100nF -> 100n
- C17: renamed from C15; value 100nF -> 100n
- C18: renamed from C16; value 100nF -> 100n
- C19: renamed from C17; value 100nF -> 100n
- C20: renamed from C18; value 100nF -> 100n
- C21: renamed from C19; value 10uF -> 10u
- C3: renamed from C1; value 15pF -> 15p
- C4: renamed from C2; value 15pF -> 15p
- C5: renamed from C3; value 100nF -> 100n
- C6: renamed from C4; value 4.7uF -> 4.7u
- C7: renamed from C5; value 4.7uF -> 4.7u
- C8: renamed from C6; value 100nF -> 100n
- C9: renamed from C7; value 4.7uF -> 4.7u
- L1: value 3.3uH -> 3.3u
- renumbered R1 to R17, R2 to R18, R3 to R19, R4 to R20, R5 to R21, R6 to R22, R7 to R23, U1 to U2, U2 to U3
Connections:
- net COL_MCU_G is gone; now on net ROW_MCU_0: U3.16 (GPIO16)
- net COL_MCU_H is gone; now on net ROW_MCU_1: U3.17 (GPIO17)
- net ROW_MCU_0: no longer U3.18 (GPIO18)
- net ROW_MCU_1: no longer U3.19 (GPIO19)
- net ROW_MCU_2: now also U3.18 (GPIO18); no longer U3.20 (GPIO20)
- net ROW_MCU_3: now also U3.19 (GPIO19); no longer U3.21 (GPIO21)
- net ROW_MCU_4: now also U3.20 (GPIO20); no longer U3.22 (GPIO22)
- net ROW_MCU_5: now also U3.21 (GPIO21); no longer U3.23 (GPIO23)
- net ROW_MCU_6: now also U3.22 (GPIO22); no longer U3.25 (GPIO24)
- net ROW_MCU_7: now also U3.23 (GPIO23); no longer U3.26 (GPIO25)
- net ROW_MCU_8: now also U3.25 (GPIO24); no longer U3.27 (GPIO26)
- net ROW_MCU_9: now also U3.26 (GPIO25); no longer U3.28 (GPIO27)
- net ROW_MCU_A: now also U3.27 (GPIO26); no longer U3.36 (GPIO28)
- net ROW_MCU_B: now also U3.28 (GPIO27); no longer U3.37 (GPIO29)
- net ROW_MCU_C: now also U3.36 (GPIO28); no longer U3.38 (GPIO30)
- net ROW_MCU_D: now also U3.37 (GPIO29); no longer U3.39 (GPIO31)
- net ROW_MCU_E: now also U3.38 (GPIO30); no longer U3.45 (GPIO36)
- net ROW_MCU_F: now also U3.39 (GPIO31); no longer U3.46 (GPIO37)
- net ROW_MCU_G: no longer names the net of U3.47 (GPIO38)
- net ROW_MCU_H: no longer names the net of U3.48 (GPIO39)
- no-connect marks 10 -> 14
Other:
- note added: "Make sure R7 and R8 are close to RP2350"
- note removed: "Make USB resistors close to RP2350"
- note removed: "Maybe use larger capacitance for 10uF capacitors (say 22uF) if using smaller package size components, e.g. 0402."
