File: panel_rp2350_18x18/layout/driver_rp2350_copy_mod.kicad_pcb (KiCad board)
At the start: 6 copper layers, 45 x 45 mm, 462 parts, among them J1 Conn_01x04, J2 Conn_01x05, J3 Conn_01x05, J4 Conn_01x05, J5 Conn_01x05, SW1 SW_Push, SW2 SW_Push, U1 APS6404L-3SQR, U10 UCC27517, U11 UCC27517, U12 UCC27517, U13 UCC27517, U14 UCC27517, U15 UCC27517, U16 UCC27517, U17 UCC27517, U18 UCC27517, U19 UCC27517, U2 RP2354B_80QFN, U20 UCC27517, U21 UCC27517, U22 UCC27517, U23 UCC27517, U24 UCC27517, U25 UCC27517, U26 UCC27517, U27 UCC27517, U28 UCC27517, U29 UCC27517, U3 UCC27517, U30 UCC27517, U31 UCC27517, U32 UCC27517, U33 UCC27517, U34 UCC27517, U35 UCC27517, U36 UCC27517, U37 UCC27517, U38 UCC27517, U39 AP2112K-3.3, U4 UCC27517, U5 UCC27517, U6 UCC27517, U7 UCC27517, U8 UCC27517, U9 UCC27517, Y1 ABM8-272-T3

Commit message: Worked on 20x20 design.
Parts:
- added C19: 10uF, Capacitor_SMD:C_0402_1005Metric, F.Cu at (-48.3, 56.8)
- C1, C10, C11, C12, C13, C14, C15, C16, C17, C18, C2, C3, C4, C5, C6, C64, C65, C7, C8, C9, L1, R1, R10, R11, R12, R13, R14, R15, R16, R17, R18, R19, R2, R20, R21, R22, R23, R24, R25, R26, R3, R4, R5, R6, R7, R8, R9, SW1, SW2, U10, U11, U12, U13, U14, U15, U16, U17, U18, U19, U20, U21, U22, U23, U24, U25, U26, U27, U28, U29, U3, U30, U31, U32, U33, U34, U35, U36, U37, U38, U39, U4, U5, U6, U7, U8, U9, Y1: moved to F.Cu
- C20: renamed from C19; moved to F.Cu
- C21: renamed from C20; moved to F.Cu
- C22: renamed from C21; moved to F.Cu
- C23: renamed from C22; moved to F.Cu
- C24: renamed from C23; moved to F.Cu
- C25: renamed from C24; moved to F.Cu
- C26: renamed from C25; moved to F.Cu
- C27: renamed from C26; moved to F.Cu
- C28: renamed from C27; moved to F.Cu
- C29: renamed from C28; moved to F.Cu
- C30: renamed from C29; moved to F.Cu
- C31: renamed from C30; moved to F.Cu
- C32: renamed from C31; moved to F.Cu
- C33: renamed from C32; moved to F.Cu
- C34: renamed from C33; moved to F.Cu
- C35: renamed from C34; moved to F.Cu
- C36: renamed from C35; moved to F.Cu
- C37: renamed from C36; moved to F.Cu
- C38: renamed from C37; moved to F.Cu
- C39: renamed from C38; moved to F.Cu
- C40: renamed from C39; moved to F.Cu
- C41: renamed from C40; moved to F.Cu
- C42: renamed from C41; moved to F.Cu
- C43: renamed from C42; moved to F.Cu
- C44: renamed from C43; moved to F.Cu
- C45: renamed from C44; moved to F.Cu
- C46: renamed from C45; moved to F.Cu
- C47: renamed from C46; moved to F.Cu
- C48: renamed from C47; moved to F.Cu
- C49: renamed from C48; moved to F.Cu
- C50: renamed from C49; moved to F.Cu
- C51: renamed from C50; moved to F.Cu
- C52: renamed from C51; moved to F.Cu
- C53: renamed from C52; moved to F.Cu
- C54: renamed from C53; moved to F.Cu
- C55: renamed from C54; moved to F.Cu
- C56: renamed from C55; moved to F.Cu
- C57: renamed from C56; moved to F.Cu
- C58: renamed from C57; moved to F.Cu
- C59: renamed from C58; moved to F.Cu
- C60: renamed from C59; moved to F.Cu
- C61: renamed from C60; moved to F.Cu
- C62: renamed from C61; moved to F.Cu
- C63: renamed from C62; moved to F.Cu
- moved R2 141.9 mm to (-43.6, 43.6), turned to 0 degrees
- moved L1 134.5 mm to (-54.8, 51.6)
- moved Y1 132.7 mm to (-59.2, 51.8)
- moved C9 131.1 mm to (-48.5, 45.3)
- moved C7 129.5 mm to (-48.3, 52.9), turned to 0 degrees
- moved C16 129.0 mm to (-46.0, 47.1)
- moved C15 128.6 mm to (-46.0, 45.3)
- moved C4 128.2 mm to (-48.3, 48.9)
- moved C14 128.1 mm to (-46.0, 43.6)
- moved C5 127.9 mm to (-48.3, 50.9)
- moved R6 126.8 mm to (-41.1, 40.1), turned to 0 degrees
- moved C3 125.7 mm to (-48.5, 41.8), turned to 0 degrees
- moved C2 125.1 mm to (-48.5, 40.1)
- moved C17 124.8 mm to (-43.6, 38.3), turned to 0 degrees
- moved C1 123.9 mm to (-48.5, 38.3), turned to 0 degrees
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Routing:
- net /panel_mcu/XIN: track 7.76 -> 0.00 mm
- net +1V1: track 4.74 -> 0.00 mm
- net /panel_mcu/VREG_LX: track 4.54 -> 0.00 mm
- net Net-(C2-Pad1): track 3.41 -> 0.00 mm
- net /panel_mcu/XOUT: track 1.77 -> 0.00 mm
- net GND: track 1.55 -> 0.00 mm
- net +3V3: track 1.55 -> 0.00 mm
- removed copper zone on B.Cu, net (none)
- removed copper zone on B.Cu, net +1V1
- removed copper zone on B.Cu, net +3V3
- removed copper zone on B.Cu, net GND
