File: panel_rp2350_20x20/manual_route/panel_rp2350_20x20_rev1.kicad_pcb (KiCad board)
At the start: 6 copper layers, 45 x 45 mm, 556 parts, among them J1 Conn_01x04, J2 Conn_01x05, J3 Conn_01x05, J4 Conn_01x05, J5 Conn_01x05, SW1 SW_Push, SW2 SW_Push, U1 APS6404L-3SQR, U10 UCC27517, U11 UCC27517, U12 UCC27517, U13 UCC27517, U14 UCC27517, U15 UCC27517, U16 UCC27517, U17 UCC27517, U18 UCC27517, U19 UCC27517, U2 RP2354B_80QFN, U20 UCC27517, U21 UCC27517, U22 UCC27517, U23 UCC27517, U24 UCC27517, U25 UCC27517, U26 UCC27517, U27 UCC27517, U28 UCC27517, U29 UCC27517, U3 UCC27517, U30 UCC27517, U31 UCC27517, U32 UCC27517, U33 UCC27517, U34 UCC27517, U35 UCC27517, U36 UCC27517, U37 UCC27517, U38 UCC27517, U39 UCC27517, U4 UCC27517, U40 UCC27517, U41 UCC27517, U42 UCC27517, U43 AP2112K-3.3, U5 UCC27517, U6 UCC27517, U7 UCC27517, U8 UCC27517, U9 UCC27517, Y1 ABM8-272-T3

Commit message: Worked on layout and routing for rp2350 20x20 panels.
Parts:
- moved C10 0.28 mm to (66.2, 78.2)
- moved C9 0.24 mm to (78.9, 76.6)
- moved C14 0.23 mm to (78.9, 72.2)
- moved C15 0.16 mm to (79.0, 75.8)
- moved C8 0.15 mm to (73.9, 69.1)
Routing:
- net /drivers/COL_MCU_04: track 5.24 -> 0.36 mm, vias 2 -> 1
- net /drivers/ROW_MCU_13: track 4.54 -> 0.01 mm, vias 2 -> 1
- net /drivers/ROW_MCU_17: track 4.46 -> 0.00 mm, vias 1 -> 0
- net /drivers/COL_MCU_00: track 4.37 -> 0.00 mm, vias 1 -> 0
- net /drivers/COL_MCU_06: track 4.37 -> 0.01 mm, vias 2 -> 1
- net /drivers/COL_MCU_12: track 4.63 -> 0.27 mm, vias 2 -> 1
- net /drivers/COL_MCU_10: track 4.65 -> 0.33 mm, vias 2 -> 1
- net /drivers/COL_MCU_05: track 4.32 -> 0.01 mm, vias 2 -> 1
- net /drivers/ROW_MCU_00: track 4.89 -> 0.78 mm, vias 2 -> 1
- net /drivers/COL_MCU_01: track 4.05 -> 0.00 mm, vias 1 -> 0
- net /drivers/COL_MCU_13: track 4.88 -> 0.89 mm, vias 2 -> 1
- net /drivers/ROW_MCU_01: track 4.29 -> 0.33 mm, vias 2 -> 1
- net /drivers/COL_MCU_15: track 3.95 -> 0.01 mm, vias 2 -> 1
- net /drivers/COL_MCU_16: track 4.78 -> 0.88 mm, vias 2 -> 1
- net /drivers/ROW_MCU_16: track 3.81 -> 0.00 mm, vias 1 -> 0
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